File: SeriesLoadLimiter_old/Programmable AC Series Limiter.sch (EAGLE design)
At the start: 67 parts, among them IC1 7805T, IC2 LM358N, IC3 LM311N, IC4 LM311N, Q1 600V 15A

Commit message: Add files via upload
Parts:
- removed IC4: LM311N, linear:LM311N
- removed JP1: (no value), jumper:JP2E
- removed R7: 3K3, resistor:R-US_0204/2V
- removed R8: 4K7, resistor:R-US_0204/2V
- removed VR3: 2K0 MT, pot:US-EVUE2A
- added D3: 1N4148, diode:1N4148DO35-7
- added Q2, Q3, Q4: BC547, transistor-npn:BC547
- added R20, R23: 4K7, resistor:R-US_0204/2V
- R19: value 1K8 -> 2K2
Connections:
- removed net N$14: IC4.ON/STR, VR3.E
- removed net N$15: IC4.ON, VR3.A
- removed net N$41: IC4.OUT, JP1.3
- removed net N$50: JP1.2, R11.2, TP3.TP
- new net N$35: Q3.C, R11.2, TP3.TP
- new net N$49: Q4.B, R23.2
- net GND: now also D3.A, Q2.E, Q3.E, Q4.E; no longer IC4.-IN, IC4.GND, R19.1
- net N$17: no longer IC4.V-
- net N$19: now also D3.C, Q2.B, R19.2; no longer R7.2, VR3.S
- net N$21: now also Q2.C, Q3.B, Q4.C, R20.2; no longer IC4.+IN, R19.2, R8.1
- net N$31: now also R19.1; no longer R8.2
- net N$46: now also R20.1; no longer IC4.V+, R7.1
- net N$47: now also R23.1; no longer JP1.1
Other:
- note removed: "Adjust for 50% duty at TP3"
- note removed: "JP1: 1-2 Test 2-3 Normal"
- moved on the sheet: R19
